File: hardware/4in1-mini.kicad_sch (KiCad schematic)
At the start: 23 parts, among them J1 SM08B-SRSS-TB, U1 TLV76733DRVR, U12 INA186A3IDCKR, U13 LMR54406DBVR, U5 FTC160808S4R7MBCA

Commit message: Rev 3: input TVS removed
The 2x SMF24A-T13 are removed. Their 24 V standoff sits below the 25.2 V a full
6S pack reaches, so they conducted rather than protected. The board stays 6S
only and now has no input clamp; DESIGN.md updated to say so.

ERC and DRC reviewed by the maintainer.

Co-Authored-By: Claude Opus 5 (1M context) <noreply@anthropic.com>
Parts:
- removed D1, D2: SMF24A-T13, 4in1ESC:SOD-123FL_L2.7-W1.8-LS3.7-RD, symbol components:SMF24A-T13
Other:
- note added: "4 to 45V, can handle 50V spikes. 1.1Mhz, 0.6A (plenty for gate driving)"
- note added: "Rev3: Removed TVS diodes, they don't start clamping until 36V or so which is already above the MOSFET voltage ratings."
- note removed: "4 to 36V, can handle 50V spikes. TBD on 8S 1.1Mhz, 0.6A (plenty for gate driving)"

Commit message: rev3.2: CSA input network against the measured high-side feedthrough
Same change as OpenESC-30x30 rev3.2: R91/R92 1k in the sense legs,
C52/C54 100n 50V to ground, C51 1u across the INA186 inputs. Worst-case
SPICE (1% R, 10% C opposed, 10 Vpp CM at 50 kHz): common-mode at the
pins down 300x, converted differential 2.8 mVpp, DC gain error -0.08
percent. Scale unchanged at 20 mV/A. Acceptance test: the ESC-04
mid-throttle i_a vs clamp sweep that convicted rev3.1
(Logs/esc-04-20x20-20260821T150430Z).

Gates G1-G6 pass with the rev3.2 baselines; fab set 20x20_ESC_Rev3.2
checked consistent against board and schematic. Silkscreen still reads
rev3.1: maintainer edit pending, fab set and renders to be regenerated
after it.

Co-Authored-By: Claude Fable 5 <noreply@anthropic.com>
Parts:
- removed Rsense1: 0.2mR, Resistor_SMD:R_2512_6332Metric, symbol Device:R
- added C51: 1uF, 4in1ESC-30x30:C_0402_1005Metric, symbol ESCLibrary:GRM033R61C104KE84D
- added C52, C54: 100nF, Capacitor_SMD:C_0402_WIDE, symbol ESCLibrary:GRM033R61C104KE84D
- added R91, R92: 1k, Capacitor_SMD:C_0201_0603Metric, symbol components:0201_1kR
- added Rsense2: 0.2mR, Resistor_SMD:R_2512_6332Metric, symbol Device:R
Connections:
- net +BATT: now also R92.2, Rsense2.2; no longer U12.5 (-IN)
- net CSA+: now also R91.2, Rsense2.1; no longer U12.4 (+IN)
- net GND: now also C52.2, C54.2
- new net: C51.1, C54.1, R92.1, U12.5 (-IN)
- new net: C51.2, C52.1, R91.1, U12.4 (+IN)
Other:
- note removed: "0.2mΩ shunt × 100V/V gain Max: 165A (3.3V ADC)"
- moved on the sheet: C93, C94, R73, U12
