File: hardware/4in1-mini.kicad_sch (KiCad schematic)
At the start: 26 parts, among them J1 SM08B-SRSS-TB, U1 TLV76733DRVR, U12 INA186A3IDCKR, U13 LMR54406DBVR, U5 FTC160808S4R7MBCA

Commit message: Fix JLCPCB placement for Q1-Q24, U12, J1 and the QFNs (#41) (#45)
The Fabrication Toolkit options enabled AUTO TRANSLATE, which applies the
toolkit's generic regex table. On this board it matched the EasyEDA-derived
QFN-24/QFN-28 footprints (+90) and SOT-23-6 (+180), which already match the
JLCPCB library orientation, and missed the parts that do differ.

Compared pad 1 and pin layout of every placed footprint against the EasyEDA
footprint of its LCSC part (easyeda2kicad):

- Q1-Q24 (C49441966): KiCad footprint is the EasyEDA one rotated 270
- U12 (C2058245): rotated 270
- J1 (C160407): same rotation, origin 2.833 mm from the EasyEDA origin
- all other placed parts: match at 0, or are two-terminal

Changes: AUTO TRANSLATE off; FT Rotation Offset 270 on Q1-Q24 and U12, FT
Position Offset 0,2.833 on J1, in the schematic symbols and the PCB
footprints. Metadata only: netlist unchanged apart from the fields, ERC 336
and DRC 68/0/184 identical before and after.

Co-authored-by: Claude Opus 5.5 <noreply@anthropic.com>
Parts:
- J1: FT Position Offset (none) -> 0,2.833
- U12: FT Rotation Offset (none) -> 270
